File: hardware/unicorder-mk-1.1.sch (EAGLE design)
At the start: 13 parts, among them IC1 TINY85

Commit message: alsdkfjkalsdf
Parts:
- removed AVR_ISP: AVR_SPI_PRG_6AVR-JST-PTH-RA-I2C, A_butts:AVR_SPI_PRG_6AVR-JST-PTH-RA-I2C
- removed BATT: M02JST-PTH-VERT, A_butts:M02JST-PTH-VERT
- removed C3: 0.1uF, A_butts:CAPACITOR-CERAMIC025-024X044
- removed IC1: TINY85, A_butts:ATTINY45TINY85-20-DIP
- removed PWR: SWITCH-SPDTPTH-RA-2MM, A_butts:SWITCH-SPDTPTH-RA-2MM
- removed R1: 10K, A_butts:RESISTORPTH-AXIAL-7.62MM
- added U1: DIGISPARK_SHIELD, A_butts:DIGISPARK_SHIELD
- DISPLAY1: value ADAFRUIT_128X64_OLED -> ADAFRUIT_128X32_OLED_I2CCLOSER; device A_butts:ADAFRUIT_128X64_OLED -> A_butts:ADAFRUIT_128X32_OLED_I2CCLOSER
Connections:
- removed net RST: AVR_ISP.RST, IC1.RESET, R1.1
- net DISPLAY_RST: now also U1.P3; no longer IC1.PB3(ADC3)
- net GND: now also U1.GND; no longer AVR_ISP.GND, BATT.1, C3.2, IC1.GND
- net MISO: now also U1.P1; no longer AVR_ISP.MISO, IC1.PB1(MISO)
- net MOSI/SDA: now also DISPLAY1.SDA, U1.P0; no longer AVR_ISP.MOSI, DISPLAY1.DATA, IC1.PB0(MOSI)
- net SCK/SCL: now also DISPLAY1.SCL, U1.P2; no longer AVR_ISP.SCK, DISPLAY1.CLK, IC1.PB2(SCK/ADC1)
- net VCC: now also U1.5V; no longer AVR_ISP.VCC, C3.1, IC1.VCC, PWR.NO, R1.2
- net V_BATT: now also U1.VIN; no longer BATT.2, PWR.COM
Other:
- moved on the sheet: C1, C2, R3
