File: hardware/unicorder-mk-1.3-base.brd (EAGLE design)
At the start: 38.2 x 32.3 mm, 13 parts, among them IC1 TINY85

Commit message: alsdkfjkalsdf
Parts:
- removed AVR_ISP: AVR_SPI_PRG_6AVR-JST-PTH-RA-I2C, A_butts:AVR-JST-6-PTH-RA-I2C
- removed BATT: M02JST-PTH-VERT, A_butts:JST-2-PH-VERT-PTH
- removed C3: 0.1uF, A_butts:C025-024X044
- removed DISPLAY1: ADAFRUIT_128X64_OLED, A_butts:ADAFRUIT_128X64_OLED
- removed IC1: TINY85, A_butts:DIP08
- removed PWR: SWITCH-SPDTPTH-RA-2MM, A_butts:SPDT-RA-2MM
- removed R1: 10K, A_butts:RESISTOR-AXIAL-PTH-7.62MM
- removed R2, R3: 4.7K, A_butts:RESISTOR-AXIAL-PTH-7.62MM
- added U1: DIGISPARK_SHIELDREV, A_butts:DIGISPARK_SHIELD_REV
- moved TSL2561 39.1 mm to (65.7, 28.6), turned to 270 degrees
- moved C1 14.3 mm to (5.29, 29.1), flipped to the bottom, turned to 180 degrees
- moved C2 8.87 mm to (20.0, 28.0), flipped to the bottom, turned to 90 degrees
- moved FRAME1 0.50 mm to (-0.60, 0.00)
Connections:
- removed net RST: AVR_ISP.RESET, IC1.1, R1.P$1
- net DISPLAY_RST: now also U1.P3; no longer DISPLAY1.RST, IC1.2
- net GND: now also U1.GND; no longer AVR_ISP.GND, BATT.1, C3.2, DISPLAY1.GND, IC1.4
- net MISO: now also U1.P1; no longer AVR_ISP.MISO, IC1.6
- net MOSI/SDA: now also U1.P0; no longer AVR_ISP.MOSI/SDA, DISPLAY1.DATA, IC1.5, R3.P$1
- net SCK/SCL: now also U1.P2; no longer AVR_ISP.SCK, DISPLAY1.CLK, IC1.7, R2.P$1
- net VCC: now also U1.5V; no longer AVR_ISP.VCC, C3.1, DISPLAY1.VIN, IC1.8, PWR.3, R1.P$2, R2.P$2, R3.P$2
- net V_BATT: now also U1.VIN; no longer BATT.2, PWR.2
Other:
- board size 38.2 x 32.3 mm -> 28 x 36 mm
