File: hardware/unicorder-mk-1.4-display.brd (EAGLE design)
At the start: 38.2 x 32.3 mm, 13 parts, among them IC1 TINY85

Commit message: alsdkfjkalsdf
Parts:
- removed AVR_ISP: AVR_SPI_PRG_6AVR-JST-PTH-RA-I2C, A_butts:AVR-JST-6-PTH-RA-I2C
- removed BATT: M02JST-PTH-VERT, A_butts:JST-2-PH-VERT-PTH
- removed C2, C3: 0.1uF, A_butts:C025-024X044
- removed IC1: TINY85, A_butts:DIP08
- removed PWR: SWITCH-SPDTPTH-RA-2MM, A_butts:SPDT-RA-2MM
- removed R1: 10K, A_butts:RESISTOR-AXIAL-PTH-7.62MM
- removed TSL2561: (no value), A_butts:1X07_PTH_SLIMASS
- added U$1: (no value), A_butts:CC-BY-SA-4.0-NO-URL
- added U$2: (no value), A_butts:COW_SMALL
- added U$3: (no value), A_butts:OSHWLOGO_TOP_0.2
- added U1: DIGISPARK_SHIELDREV, A_butts:DIGISPARK_SHIELD_REV
- added U2: ADAFRUIT_TSL2561, A_butts:ADAFRUIT_TSL2561
- DISPLAY1: value ADAFRUIT_128X64_OLED -> ADAFRUIT_128X32_OLED_I2CNOSILK_NOHOLES_NOPROBLEM; device A_butts:ADAFRUIT_128X64_OLED -> A_butts:ADAFRUIT_128X32_OLED_I2C_CLOSER_NS
- moved DISPLAY1 26.1 mm to (8.10, 1.85)
- moved R2 23.4 mm to (7.90, 5.00), flipped to the bottom, turned to 180 degrees
- moved R3 19.7 mm to (7.90, 7.56), flipped to the bottom, turned to 180 degrees
- moved C1 14.0 mm to (14.4, 6.29), flipped to the bottom, turned to 90 degrees
Connections:
- removed net RST: AVR_ISP.RESET, IC1.1, R1.P$1
- net DISPLAY_RST: now also U1.P3; no longer IC1.2
- net GND: now also U1.GND, U2.GND; no longer AVR_ISP.GND, BATT.1, C2.2, C3.2, IC1.4, TSL2561.6
- net MISO: now also U1.P1; no longer AVR_ISP.MISO, IC1.6
- net MOSI/SDA: now also DISPLAY1.SDA, U1.P0, U2.SDA; no longer AVR_ISP.MOSI/SDA, DISPLAY1.DATA, IC1.5, TSL2561.2
- net SCK/SCL: now also DISPLAY1.SCL, U1.P2, U2.SCL; no longer AVR_ISP.SCK, DISPLAY1.CLK, IC1.7, TSL2561.1
- net VCC: now also U1.5V, U2.VIN; no longer AVR_ISP.VCC, C2.1, C3.1, IC1.8, PWR.3, R1.P$2, TSL2561.7
- net V_BATT: now also U1.VIN; no longer BATT.2, PWR.2
Routing:
- net VCC: track 0.00 -> 41.9 mm
- net MOSI/SDA: track 0.00 -> 37.0 mm
- net SCK/SCL: track 0.00 -> 29.0 mm
- net DISPLAY_RST: track 0.00 -> 17.2 mm
Other:
- board size 38.2 x 32.3 mm -> 19.2 x 24 mm
- board text added: ">VERSION"
- board text added: "I2C Disp"
- board text added: "TSL2561 Lux Sensor"
- board text added: "WHAT THE LUX?"
- board text added: "by schizobovine <sean@yak.net>"
