File: hardware/unicorder-mk-2.0.sch (EAGLE design)
At the start: 13 parts, among them IC1 TINY85

Commit message: alsdkfjkalsdf
Parts:
- removed AVR_ISP: AVR_SPI_PRG_6AVR-JST-PTH-RA-I2C, A_butts:AVR_SPI_PRG_6AVR-JST-PTH-RA-I2C
- removed C3: 0.1uF, A_butts:CAPACITOR-CERAMIC025-024X044
- removed IC1: TINY85, A_butts:ATTINY45TINY85-20-DIP
- removed R1: 10K, A_butts:RESISTORPTH-AXIAL-7.62MM
- added SHIELD: (no value), A_butts:ARDUINO_SHIELD_SMALLER
- DISPLAY1: value ADAFRUIT_128X64_OLED -> ADAFRUIT_128X64_OLEDCLOSER; device A_butts:ADAFRUIT_128X64_OLED -> A_butts:ADAFRUIT_128X64_OLEDCLOSER
- R2, R3: device A_butts:RESISTORPTH-AXIAL-7.62MM -> A_butts:RESISTORPTH-AXIAL-5.08MM
Connections:
- removed net MISO: AVR_ISP.MISO, IC1.PB1(MISO)
- removed net RST: AVR_ISP.RST, IC1.RESET, R1.1
- net DISPLAY_RST: no longer IC1.PB3(ADC3)
- net GND: no longer AVR_ISP.GND, C3.2, IC1.GND
- net MOSI/SDA: no longer AVR_ISP.MOSI, IC1.PB0(MOSI)
- net SCK/SCL: no longer AVR_ISP.SCK, IC1.PB2(SCK/ADC1)
- net VCC: no longer AVR_ISP.VCC, C3.1, IC1.VCC, R1.2
Changed lines of the file:
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@@
 <part name="GND1" library="A_butts" deviceset="GND" device=""/>
 <part name="SUPPLY1" library="A_butts" deviceset="VCC" device=""/>
-<part name="IC1" library="A_butts" deviceset="ATTINY45" device="TINY85-20-DIP" value="TINY85"/>
 <part name="C1" library="A_butts" deviceset="CAPACITOR-CERAMIC" device="025-024X044" value="0.1uF"/>
 <part name="C2" library="A_butts" deviceset="CAPACITOR-CERAMIC" device="025-024X044" value="0.1uF"/>
-<part name="C3" library="A_butts" deviceset="CAPACITOR-CERAMIC" device="025-024X044" value="0.1uF"/>
-<part name="R1" library="A_butts" deviceset="RESISTOR" device="PTH-AXIAL-7.62MM" value="10K"/>
-<part name="AVR_ISP" library="A_butts" deviceset="AVR_SPI_PRG_6" device="AVR-JST-PTH-RA-I2C" value="AVR_SPI_PRG_6AVR-JST-PTH-RA-I2C"/>
-<part name="SUPPLY2" library="A_butts" deviceset="VCC" device=""/>
-<part name="GND2" library="A_butts" deviceset="GND" device=""/>
-<part name="SUPPLY3" library="A_butts" deviceset="VCC" device=""/>
-<part name="R2" library="A_butts" deviceset="RESISTOR" device="PTH-AXIAL-7.62MM" value="4.7K"/>
-<part name="R3" library="A_butts" deviceset="RESISTOR" device="PTH-AXIAL-7.62MM" value="4.7K"/>
+<part name="R2" library="A_butts" deviceset="RESISTOR" device="PTH-AXIAL-5.08MM" value="4.7K"/>
+<part name="R3" library="A_butts" deviceset="RESISTOR" device="PTH-AXIAL-5.08MM" value="4.7K"/>
 <part name="SUPPLY4" library="A_butts" deviceset="VCC" device=""/>
 <part name="SUPPLY5" library="A_butts" deviceset="VCC" device=""/>
-<part name="DISPLAY1" library="A_butts" deviceset="ADAFRUIT_128X64_OLED" device=""/>
+<part name="DISPLAY1" library="A_butts" deviceset="ADAFRUIT_128X64_OLED" device="CLOSER" value="ADAFRUIT_128X64_OLEDCLOSER"/>
 <part name="SUPPLY6" library="A_butts" deviceset="VCC" device=""/>
 <part name="GND3" library="A_butts" deviceset="GND" device=""/>
 <part name="SUPPLY7" library="A_butts" deviceset="VCC" device=""/>
 <part name="GND4" library="A_butts" deviceset="GND" device=""/>
-<part name="GND5" library="A_butts" deviceset="GND" device=""/>
-<part name="SUPPLY8" library="A_butts" deviceset="VCC" device=""/>
 <part name="BATT" library="A_butts" deviceset="M02" device="JST-PTH-VERT"/>
 <part name="PWR" library="A_butts" deviceset="SWITCH-SPDT" device="PTH-RA-2MM"/>
@@
 <part name="SUPPLY12" library="A_butts" deviceset="V_BATT" device=""/>
 <part name="GND8" library="A_butts" deviceset="GND" device=""/>
+<part name="SHIELD" library="A_butts" deviceset="ARDUINO_SHIELD_SMALLER" device=""/>
 </parts>
 <sheets>
@@
 <instance part="GND1" gate="1" x="139.7" y="111.76"/>
 <instance part="SUPPLY1" gate="G$1" x="139.7" y="134.62"/>
-<instance part="IC1" gate="G$1" x="157.48" y="124.46"/>
 <instance part="C1" gate="G$1" x="139.7" y="124.46" rot="MR0"/>
 <instance part="C2" gate="G$1" x="63.5" y="162.56"/>
-<instance part="C3" gate="G$1" x="137.16" y="162.56"/>
-<instance part="R1" gate="G$1" x="175.26" y="139.7" rot="R90"/>
-<instance part="AVR_ISP" gate="G$1" x="147.32" y="83.82"/>
-<instance part="SUPPLY2" gate="G$1" x="160.02" y="88.9"/>
-<instance part="GND2" gate="1" x="160.02" y="76.2"/>
-<instance part="SUPPLY3" gate="G$1" x="175.26" y="147.32"/>
 <instance part="R2" gate="G$1" x="200.66" y="144.78" rot="R90"/>
 <instance part="R3" gate="G$1" x="208.28" y="144.78" rot="R90"/>
@@
 <instance part="SUPPLY6" gate="G$1" x="25.4" y="172.72"/>
 <instance part="GND3" gate="1" x="25.4" y="144.78"/>
-<instance part="SUPPLY7" gate="G$1" x="63.5" y="167.64"/>
-<instance part="GND4" gate="1" x="63.5" y="154.94"/>
-<instance part="GND5" gate="1" x="137.16" y="154.94"/>
-<instance part="SUPPLY8" gate="G$1" x="137.16" y="167.64"/>
+<instance part="SUPPLY7" gate="G$1" x="63.5" y="170.18"/>
+<instance part="GND4" gate="1" x="63.5" y="152.4"/>
 <instance part="BATT" gate="G$1" x="20.32" y="119.38"/>
 <instance part="PWR" gate="G$1" x="43.18" y="124.46" rot="MR180"/>
@@
 <instance part="SUPPLY12" gate="G$1" x="22.86" y="104.14"/>
 <instance part="GND8" gate="1" x="22.86" y="86.36"/>
+<instance part="SHIELD" gate="G$1" x="71.12" y="78.74"/>
 </instances>
 <busses>
@@
 <segment>
 <pinref part="SUPPLY1" gate="G$1" pin="VCC"/>
-<wire x1="139.7" y1="134.62" x2="139.7" y2="132.08" width="0.1524" layer="91"/>
-<pinref part="IC1" gate="G$1" pin="VCC"/>
-<wire x1="139.7" y1="132.08" x2="142.24" y2="132.08" width="0.1524" layer="91"/>
 <pinref part="C1" gate="G$1" pin="1"/>
-<wire x1="139.7" y1="129.54" x2="139.7" y2="132.08" width="0.1524" layer="91"/>
-<junction x="139.7" y="132.08"/>
-</segment>
-<segment>
-<pinref part="AVR_ISP" gate="G$1" pin="VCC"/>
-<wire x1="157.48" y1="86.36" x2="160.02" y2="86.36" width="0.1524" layer="91"/>
-<pinref part="SUPPLY2" gate="G$1" pin="VCC"/>
-<wire x1="160.02" y1="86.36" x2="160.02" y2="88.9" width="0.1524" layer="91"/>
-</segment>
-<segment>
-<pinref part="R1" gate="G$1" pin="2"/>
-<pinref part="SUPPLY3" gate="G$1" pin="VCC"/>
-<wire x1="175.26" y1="147.32" x2="175.26" y2="144.78" width="0.1524" layer="91"/>
+<wire x1="139.7" y1="129.54" x2="139.7" y2="134.62" width="0.1524" layer="91"/>
 </segment>
 <segment>
@@
 <pinref part="C2" gate="G$1" pin="1"/>
 <pinref part="SUPPLY7" gate="G$1" pin="VCC"/>
-</segment>
-<segment>
-<pinref part="C3" gate="G$1" pin="1"/>
-<pinref part="SUPPLY8" gate="G$1" pin="VCC"/>
+<wire x1="63.5" y1="170.18" x2="63.5" y2="167.64" width="0.1524" layer="91"/>
 </segment>
 <segment>
@@
 <segment>
 <pinref part="C1" gate="G$1" pin="2"/>
-<wire x1="139.7" y1="119.38" x2="139.7" y2="116.84" width="0.1524" layer="91"/>
-<pinref part="IC1" gate="G$1" pin="GND"/>
-<wire x1="139.7" y1="116.84" x2="142.24" y2="116.84" width="0.1524" layer="91"/>
 <pinref part="GND1" gate="1" pin="GND"/>
-<wire x1="139.7" y1="114.3" x2="139.7" y2="116.84" width="0.1524" layer="91"/>
-<junction x="139.7" y="116.84"/>
-</segment>
-<segment>
-<pinref part="AVR_ISP" gate="G$1" pin="GND"/>
-<wire x1="157.48" y1="81.28" x2="160.02" y2="81.28" width="0.1524" layer="91"/>
-<pinref part="GND2" gate="1" pin="GND"/>
-<wire x1="160.02" y1="81.28" x2="160.02" y2="78.74" width="0.1524" layer="91"/>
+<wire x1="139.7" y1="114.3" x2="139.7" y2="119.38" width="0.1524" layer="91"/>
 </segment>
 <segment>
@@
 <pinref part="C2" gate="G$1" pin="2"/>
 <pinref part="GND4" gate="1" pin="GND"/>
-</segment>
-<segment>
-<pinref part="C3" gate="G$1" pin="2"/>
-<pinref part="GND5" gate="1" pin="GND"/>
+<wire x1="63.5" y1="154.94" x2="63.5" y2="157.48" width="0.1524" layer="91"/>
 </segment>
 <segment>
@@
 <net name="MOSI/SDA" class="0">
 <segment>
-<pinref part="AVR_ISP" gate="G$1" pin="MOSI"/>
-<wire x1="160.02" y1="83.82" x2="157.48" y2="83.82" width="0.1524" layer="91"/>
-<label x="160.02" y="83.82" size="1.27" layer="95" xref="yes"/>
-</segment>
-<segment>
-<wire x1="175.26" y1="127" x2="172.72" y2="127" width="0.1524" layer="91"/>
-<label x="175.26" y="127" size="1.27" layer="95" xref="yes"/>
-<pinref part="IC1" gate="G$1" pin="PB0(MOSI)"/>
-</segment>
-<segment>
 <wire x1="208.28" y1="137.16" x2="208.28" y2="139.7" width="0.1524" layer="91"/>
 <label x="208.28" y="137.16" size="1.27" layer="95" rot="R270" xref="yes"/>
@@
 </segment>
 </net>
-<net name="RST" class="0">
-<segment>
-<pinref part="AVR_ISP" gate="G$1" pin="RST"/>
-<wire x1="134.62" y1="81.28" x2="137.16" y2="81.28" width="0.1524" layer="91"/>
-<label x="134.62" y="81.28" size="1.27" layer="95" rot="R180" xref="yes"/>
-</segment>
-<segment>
-<wire x1="177.8" y1="132.08" x2="175.26" y2="132.08" width="0.1524" layer="91"/>
-<label x="177.8" y="132.08" size="1.27" layer="95" rot="MR180" xref="yes"/>
-<pinref part="IC1" gate="G$1" pin="RESET"/>
-<pinref part="R1" gate="G$1" pin="1"/>
-<wire x1="175.26" y1="132.08" x2="172.72" y2="132.08" width="0.1524" layer="91"/>
-<wire x1="175.26" y1="132.08" x2="175.26" y2="134.62" width="0.1524" layer="91"/>
-<junction x="175.26" y="132.08"/>
-</segment>
-</net>
 <net name="SCK/SCL" class="0">
-<segment>
-<pinref part="AVR_ISP" gate="G$1" pin="SCK"/>
-<wire x1="134.62" y1="83.82" x2="137.16" y2="83.82" width="0.1524" layer="91"/>
-<label x="134.62" y="83.82" size="1.27" layer="95" rot="R180" xref="yes"/>
-</segment>
-<segment>
-<wire x1="175.26" y1="121.92" x2="172.72" y2="121.92" width="0.1524" layer="91"/>
-<label x="175.26" y="121.92" size="1.27" layer="95" rot="MR180" xref="yes"/>
-<pinref part="IC1" gate="G$1" pin="PB2(SCK/ADC1)"/>
-</segment>
 <segment>
 <wire x1="200.66" y1="137.16" x2="200.66" y2="139.7" width="0.1524" layer="91"/>
@@
 </segment>
 </net>
-<net name="MISO" class="0">
-<segment>
-<pinref part="AVR_ISP" gate="G$1" pin="MISO"/>
-<wire x1="134.62" y1="86.36" x2="137.16" y2="86.36" width="0.1524" layer="91"/>
-<label x="134.62" y="86.36" size="1.27" layer="95" rot="R180" xref="yes"/>
-</segment>
-<segment>
-<wire x1="175.26" y1="124.46" x2="172.72" y2="124.46" width="0.1524" layer="91"/>
-<label x="175.26" y="124.46" size="1.27" layer="95" rot="MR180" xref="yes"/>
-<pinref part="IC1" gate="G$1" pin="PB1(MISO)"/>
-</segment>
-</net>
 <net name="DISPLAY_RST" class="0">
 <segment>
-<pinref part="IC1" gate="G$1" pin="PB3(ADC3)"/>
-<wire x1="175.26" y1="119.38" x2="172.72" y2="119.38" width="0.1524" layer="91"/>
-<label x="175.26" y="119.38" size="1.27" layer="95" xref="yes"/>
-</segment>
-<segment>
 <pinref part="DISPLAY1" gate="G$1" pin="RST"/>
